File: PCB.brd (EAGLE design)
At the start: 127 x 44.5 mm, 43 parts, among them IC1 PIC16F1826/27SO, IC2 MAX3467CPA, U1 +12v, Y1 ASL-16.000MHZ-L-C-S-50-T

Commit message: Real HW R1
Parts:
- X4: device con-subd:M09H -> con-subd:F09HP
- turned X4 to 0 degrees
Routing:
- net VCC: track 118.8 -> 143.1 mm
- net RXN: track 21.7 -> 29.4 mm
- net RXP: track 14.9 -> 21.1 mm
- net TXN: track 23.9 -> 30.1 mm
- net TXP: track 23.1 -> 26.1 mm
Changed lines of the file:
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@@
 <attribute name="NAME" x="103.551" y="25.2175" size="0.8128" layer="25" font="fixed" ratio="20" align="bottom-center"/>
 </element>
-<element name="X4" library="con-subd" package="M09H" value="" x="111.125" y="33.02" smashed="yes" rot="R180">
-<attribute name="OC_FARNELL" value="unknown" x="111.125" y="33.02" size="1.778" layer="27" rot="R180" display="off"/>
-<attribute name="MPN" value="" x="111.125" y="33.02" size="1.778" layer="27" rot="R180" display="off"/>
-<attribute name="MF" value="" x="111.125" y="33.02" size="1.778" layer="27" rot="R180" display="off"/>
-<attribute name="OC_NEWARK" value="unknown" x="111.125" y="33.02" size="1.778" layer="27" rot="R180" display="off"/>
-<attribute name="VALUE" x="116.205" y="19.05" size="1.778" layer="27" ratio="10" rot="R180"/>
+<element name="X4" library="con-subd" package="F09HP" value="" x="111.125" y="33.02" smashed="yes">
+<attribute name="OC_FARNELL" value="unknown" x="111.125" y="33.02" size="1.778" layer="27" display="off"/>
+<attribute name="MPN" value="" x="111.125" y="33.02" size="1.778" layer="27" display="off"/>
+<attribute name="MF" value="" x="111.125" y="33.02" size="1.778" layer="27" display="off"/>
+<attribute name="OC_NEWARK" value="unknown" x="111.125" y="33.02" size="1.778" layer="27" display="off"/>
+<attribute name="VALUE" x="106.045" y="46.99" size="1.778" layer="27" ratio="10"/>
 </element>
 <element name="U1" library="SparkFun-IC-Power" package="TO-252" value="+12v" x="5.08" y="21.59" smashed="yes" rot="MR0">
@@
 <wire x1="99.565" y1="27.94" x2="99.695" y2="27.94" width="1.016" layer="16"/>
 <wire x1="99.695" y1="27.94" x2="89.535" y2="27.94" width="1.016" layer="1"/>
-<wire x1="107.0102" y1="34.29" x2="115.7" y2="38.1" width="0" layer="19" extent="16-16"/>
-<wire x1="105.6386" y1="31.75" x2="107.0102" y2="34.29" width="0" layer="19" extent="1-1"/>
-<wire x1="102.87" y1="29.21" x2="105.6386" y2="31.75" width="0" layer="19" extent="1-1"/>
+<wire x1="115.2398" y1="34.29" x2="115.2398" y2="33.1216" width="1.016" layer="1"/>
+<wire x1="115.2398" y1="33.1216" x2="116.6114" y2="31.75" width="1.016" layer="1"/>
+<wire x1="115.2398" y1="34.29" x2="115.2398" y2="35.8902" width="1.016" layer="1"/>
+<wire x1="115.2398" y1="35.8902" x2="114.3" y2="36.83" width="1.016" layer="1"/>
+<wire x1="114.3" y1="36.83" x2="104.14" y2="36.83" width="1.016" layer="1"/>
+<wire x1="104.14" y1="36.83" x2="102.87" y2="35.56" width="1.016" layer="1"/>
+<wire x1="102.87" y1="35.56" x2="102.87" y2="29.21" width="1.016" layer="1"/>
+<wire x1="114.3" y1="36.83" x2="115.7" y2="38.1" width="0" layer="19" extent="1-16"/>
 </signal>
 <signal name="SCK">
@@
 <wire x1="116.84" y1="26.67" x2="116.205" y2="27.305" width="0.3048" layer="16"/>
 <wire x1="116.205" y1="27.305" x2="112.8268" y2="27.305" width="0.3048" layer="16"/>
-<wire x1="112.8268" y1="27.305" x2="113.8682" y2="31.75" width="0" layer="19" extent="16-16"/>
+<wire x1="108.3818" y1="31.75" x2="112.8268" y2="27.305" width="0.3048" layer="16"/>
 </signal>
 <signal name="RXN">
@@
 <wire x1="122.4534" y1="17.145" x2="121.0564" y2="17.145" width="0.3048" layer="1"/>
 <wire x1="121.0564" y1="17.145" x2="120.4214" y2="17.78" width="0.3048" layer="1"/>
-<wire x1="113.03" y1="27.94" x2="112.4966" y2="34.29" width="0" layer="19" extent="16-16"/>
+<wire x1="109.7534" y1="34.29" x2="109.7534" y2="31.2166" width="0.3048" layer="16"/>
+<wire x1="109.7534" y1="31.2166" x2="113.03" y2="27.94" width="0.3048" layer="16"/>
 </signal>
 <signal name="TXN">
@@
 <wire x1="122.4534" y1="15.875" x2="121.0564" y2="15.875" width="0.3048" layer="1"/>
 <wire x1="121.0564" y1="15.875" x2="120.4214" y2="15.24" width="0.3048" layer="1"/>
-<wire x1="113.665" y1="28.575" x2="109.7534" y2="34.29" width="0" layer="19" extent="16-16"/>
+<wire x1="112.4966" y1="34.29" x2="112.4966" y2="29.7434" width="0.3048" layer="16"/>
+<wire x1="112.4966" y1="29.7434" x2="113.665" y2="28.575" width="0.3048" layer="16"/>
 </signal>
 <signal name="TXP">
@@
 <via x="118.11" y="29.21" extent="1-16" drill="0.5"/>
 <wire x1="118.11" y1="29.21" x2="114.935" y2="29.21" width="0.3048" layer="16"/>
-<wire x1="114.935" y1="29.21" x2="108.3818" y2="31.75" width="0" layer="19" extent="16-16"/>
+<wire x1="113.8682" y1="31.75" x2="113.8682" y2="30.2768" width="0.3048" layer="16"/>
+<wire x1="113.8682" y1="30.2768" x2="114.935" y2="29.21" width="0.3048" layer="16"/>
 </signal>
 <signal name="N$29">
