File: PCB.sch (EAGLE design)
At the start: 43 parts, among them IC1 PIC16F1826/27SO, IC2 MAX3467CPA, U1 +12v, Y1 ASL-16.000MHZ-L-C-S-50-T

Commit message: Real HW R1
Parts:
- X4: device con-subd:M09H -> con-subd:F09HP
Changed lines of the file:
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@@
 <part name="Y1" library="SparkFun-Clocks" deviceset="OSCILLATOR" device="SMD-7X5-4PAD" value="ASL-16.000MHZ-L-C-S-50-T"/>
 <part name="SUPPLY42" library="supply2" deviceset="+5V" device=""/>
-<part name="X4" library="con-subd" deviceset="M09" device="H"/>
+<part name="X4" library="con-subd" deviceset="F09" device="HP"/>
 <part name="SUPPLY43" library="supply2" deviceset="GND" device=""/>
 <part name="SUPPLY44" library="supply2" deviceset="GND" device=""/>
@@
 <instance part="Y1" gate="G$1" x="-33.02" y="68.58"/>
 <instance part="SUPPLY42" gate="+5V" x="-45.72" y="73.66"/>
-<instance part="X4" gate="-1" x="-104.14" y="30.48"/>
-<instance part="SUPPLY43" gate="GND" x="-93.98" y="35.56" rot="R90"/>
-<instance part="SUPPLY44" gate="GND" x="-114.3" y="35.56" rot="R270"/>
-<instance part="SUPPLY45" gate="G$1" x="-93.98" y="25.4" rot="R270"/>
-<instance part="SUPPLY46" gate="G$1" x="-114.3" y="27.94" rot="R90"/>
+<instance part="X4" gate="G$1" x="-106.68" y="30.48"/>
+<instance part="SUPPLY43" gate="GND" x="-116.84" y="35.56" rot="R270"/>
+<instance part="SUPPLY44" gate="GND" x="-96.52" y="33.02" rot="R90"/>
+<instance part="SUPPLY45" gate="G$1" x="-116.84" y="25.4" rot="R90"/>
+<instance part="SUPPLY46" gate="G$1" x="-96.52" y="25.4" rot="R270"/>
 <instance part="SUPPLY47" gate="+5V" x="7.62" y="109.22"/>
 <instance part="SUPPLY48" gate="GND" x="-15.24" y="96.52"/>
@@
 </segment>
 <segment>
-<pinref part="X4" gate="-1" pin="1"/>
+<pinref part="X4" gate="G$1" pin="1"/>
 <pinref part="SUPPLY43" gate="GND" pin="GND"/>
 </segment>
 <segment>
-<pinref part="X4" gate="-1" pin="6"/>
+<pinref part="X4" gate="G$1" pin="6"/>
 <pinref part="SUPPLY44" gate="GND" pin="GND"/>
 </segment>
@@
 </segment>
 <segment>
-<pinref part="X4" gate="-1" pin="5"/>
+<pinref part="X4" gate="G$1" pin="5"/>
 <pinref part="SUPPLY45" gate="G$1" pin="VCC"/>
 </segment>
 <segment>
-<pinref part="X4" gate="-1" pin="9"/>
+<pinref part="X4" gate="G$1" pin="9"/>
 <pinref part="SUPPLY46" gate="G$1" pin="VCC"/>
 </segment>
@@
 <pinref part="IC2" gate="G$1" pin="A"/>
 <wire x1="-73.66" y1="25.4" x2="-91.44" y2="25.4" width="0.1524" layer="91"/>
-<wire x1="-91.44" y1="25.4" x2="-91.44" y2="33.02" width="0.1524" layer="91"/>
-<pinref part="X4" gate="-1" pin="2"/>
-<wire x1="-91.44" y1="33.02" x2="-96.52" y2="33.02" width="0.1524" layer="91"/>
+<wire x1="-91.44" y1="25.4" x2="-91.44" y2="40.64" width="0.1524" layer="91"/>
+<pinref part="X4" gate="G$1" pin="2"/>
+<wire x1="-91.44" y1="40.64" x2="-121.92" y2="40.64" width="0.1524" layer="91"/>
+<wire x1="-121.92" y1="40.64" x2="-121.92" y2="33.02" width="0.1524" layer="91"/>
+<wire x1="-121.92" y1="33.02" x2="-114.3" y2="33.02" width="0.1524" layer="91"/>
 </segment>
 </net>
@@
 <pinref part="IC2" gate="G$1" pin="B"/>
 <wire x1="-73.66" y1="20.32" x2="-88.9" y2="20.32" width="0.1524" layer="91"/>
-<pinref part="X4" gate="-1" pin="7"/>
+<pinref part="X4" gate="G$1" pin="7"/>
 <pinref part="JP2" gate="G$1" pin="1"/>
 <wire x1="-68.58" y1="55.88" x2="-88.9" y2="55.88" width="0.1524" layer="91"/>
-<wire x1="-88.9" y1="55.88" x2="-88.9" y2="40.64" width="0.1524" layer="91"/>
-<wire x1="-88.9" y1="40.64" x2="-88.9" y2="20.32" width="0.1524" layer="91"/>
-<wire x1="-111.76" y1="33.02" x2="-121.92" y2="33.02" width="0.1524" layer="91"/>
-<wire x1="-121.92" y1="33.02" x2="-121.92" y2="40.64" width="0.1524" layer="91"/>
-<wire x1="-121.92" y1="40.64" x2="-88.9" y2="40.64" width="0.1524" layer="91"/>
-<junction x="-88.9" y="40.64"/>
+<wire x1="-88.9" y1="55.88" x2="-88.9" y2="30.48" width="0.1524" layer="91"/>
+<wire x1="-88.9" y1="30.48" x2="-88.9" y2="20.32" width="0.1524" layer="91"/>
+<wire x1="-99.06" y1="30.48" x2="-88.9" y2="30.48" width="0.1524" layer="91"/>
+<junction x="-88.9" y="30.48"/>
 </segment>
 </net>
@@
 <pinref part="IC2" gate="G$1" pin="Z"/>
 <wire x1="-73.66" y1="30.48" x2="-81.28" y2="30.48" width="0.1524" layer="91"/>
-<pinref part="X4" gate="-1" pin="8"/>
+<pinref part="X4" gate="G$1" pin="8"/>
 <pinref part="JP1" gate="G$1" pin="1"/>
 <wire x1="-68.58" y1="66.04" x2="-81.28" y2="66.04" width="0.1524" layer="91"/>
-<wire x1="-81.28" y1="66.04" x2="-81.28" y2="43.18" width="0.1524" layer="91"/>
-<wire x1="-81.28" y1="43.18" x2="-81.28" y2="30.48" width="0.1524" layer="91"/>
-<wire x1="-111.76" y1="30.48" x2="-124.46" y2="30.48" width="0.1524" layer="91"/>
-<wire x1="-124.46" y1="30.48" x2="-124.46" y2="43.18" width="0.1524" layer="91"/>
-<wire x1="-124.46" y1="43.18" x2="-81.28" y2="43.18" width="0.1524" layer="91"/>
-<junction x="-81.28" y="43.18"/>
+<wire x1="-81.28" y1="66.04" x2="-81.28" y2="30.48" width="0.1524" layer="91"/>
+<wire x1="-99.06" y1="27.94" x2="-81.28" y2="27.94" width="0.1524" layer="91"/>
+<wire x1="-81.28" y1="27.94" x2="-81.28" y2="30.48" width="0.1524" layer="91"/>
+<junction x="-81.28" y="30.48"/>
 </segment>
 </net>
@@
 <segment>
 <pinref part="IC2" gate="G$1" pin="Y"/>
-<wire x1="-73.66" y1="35.56" x2="-86.36" y2="35.56" width="0.1524" layer="91"/>
-<wire x1="-86.36" y1="35.56" x2="-86.36" y2="27.94" width="0.1524" layer="91"/>
-<pinref part="X4" gate="-1" pin="4"/>
-<wire x1="-86.36" y1="27.94" x2="-96.52" y2="27.94" width="0.1524" layer="91"/>
-</segment>
-</net>
+<wire x1="-73.66" y1="35.56" x2="-83.82" y2="35.56" width="0.1524" layer="91"/>
+<wire x1="-83.82" y1="35.56" x2="-83.82" y2="43.18" width="0.1524" layer="91"/>
+<pinref part="X4" gate="G$1" pin="4"/>
+<wire x1="-83.82" y1="43.18" x2="-124.46" y2="43.18" width="0.1524" layer="91"/>
+<wire x1="-124.46" y1="43.18" x2="-124.46" y2="27.94" width="0.1524" layer="91"/>
+<wire x1="-124.46" y1="27.94" x2="-114.3" y2="27.94" width="0.1524" layer="91"/>
+</segment>
+</net>
