File: PCB.sch (EAGLE design)
At the start: 45 parts, among them IC1 PIC16F1826/27SO, IC2 MAX3467CPA, U1 +12v, Y1 ASL-16.000MHZ-L-C-S-50-T

Commit message: Updating PCB design
Parts:
- removed IC2: MAX3467CPA, maxim:MAX3467CPA
- removed J1: (no value), SparkFun-Connectors:CONN_08"
- removed J2: (no value), SparkFun-Connectors:CONN_01
- removed JP1, JP2, JP3, JP4, JP5: JUMPER-SMT_2_NO_NO-SILK, SparkFun-Jumpers:JUMPER-SMT_2_NO_NO-SILK
- removed R10, R12, R14, R15: (no value), resistor:R-US_M1206
- removed TP3: PTR1B1,27, testpad:PTR1B1,27
- removed X1, X2, X3: (no value), con-subd:F09HP
- removed X4: (no value), con-subd:M09H
- added 5V@1, 5V@2, 5V@3, GND@1, GND@2, GND@3, GND@4, GND@5, GND@6, M1!C1, M1!C2, M1C1, M1C2, M2!C1, M2!C2, M2C1, M2C2, M3!C1, M3!C2, M3C1, M3C2, REFL1, REFL2, REFL3, REFR1, REFR2, REFR3, RX, TS1, TS2, TS3, TS4, TS5, TS6, TSCOM@1, TSCOM@2, TSCOM@3, TSCOM@4, TSCOM@5, TX, VCC@1, VCC@2, VCC@3: WIREPADSMD2,54-5,08, wirepad:WIREPADSMD2,54-5,08
- added DBGSER: (no value), SparkFun-Connectors:CONN_03
- added U2: PIC18F47Q84, FRC696:PIC18F47Q84
- C3, C5: value (none) -> 0.1uF
- C4, C6: value (none) -> 1uF
- IC1: value PIC16F1826/27SO -> LM393D; device microchip:PIC16F1826/27SO -> linear:LM393D
- PROG: value 53047-05 -> PIC-PROG047; device con-molex:53047-05 -> FRC696:PIC-PROG047
- R1, R11, R2, R3, R5, R7, R9: value (none) -> 5k
- R13: value (none) -> 330
- R4, R6: value (none) -> 10k
- R8: value (none) -> 2.2k
Connections:
- removed net N$25: IC1.RA7, TP3.TP
- removed net N$29: DRV2.VIO, JP4.1
- removed net N$30: DRV1.VIO, JP3.1
- removed net N$31: DRV3.VIO, JP5.1
- removed net N$33: IC1.RA2, R14.1, R15.2
- removed net RXN: IC2.B, JP2.1, X4.8
- removed net RXP: IC2.A, X4.4
- removed net TXN: IC2.Z, JP1.1, X4.7
- removed net TXP: IC2.Y, X4.2
- new net DBGRX: DBGSER.3, U2.RC3
- new net DBGTX: DBGSER.2, U2.RC2
- new net N$26: IC1A.-IN, R6.1, R8.2
- new net REFL1P: R1.2, U2.RB0
- new net REFL2P: R5.2, U2.RB1
- new net REFL3P: R9.2, U2.RB2
- new net REFR1P: R3.2, U2.RB3
- new net REFR2P: R7.2, U2.RB4
- new net REFR3P: R11.2, U2.RB5
- new net TS1: TS1.P, U2.RA2
- new net TS2: TS2.P, U2.RA1
- new net TS3: TS3.P, U2.RA0
- new net TS4: TS4.P, U2.RA3
- new net TS5: TS5.P, U2.RA4
- new net TS6: TS6.P, U2.RA5
- new net TSCOM: IC1A.+IN, R4.2, TSCOM@1.P, TSCOM@2.P, TSCOM@3.P, TSCOM@4.P, TSCOM@5.P
- new net TSOUT: IC1A.OUT
- net +5V: now also 5V@1.P, 5V@2.P, 5V@3.P, DRV1.VIO, DRV2.VIO, DRV3.VIO, IC1P.V+, PROGVDD.S, R2.2, R6.2, U2.VDD@1, U2.VDD@2; no longer IC1.VDD, IC2.VCC, JP3.2, JP4.2, JP5.2, PROG-2.S, R1.2, R11.2, R3.2, R5.2, R7.2, R9.2, X1.5, X2.5, X3.5
- net D1CS: now also U2.RC4; no longer IC1.RA3, J1.3
- net D2CS: now also U2.RD5; no longer IC1.RB0, J1.5
- net D3CS: now also U2.RD6; no longer IC1.RA4, J1.4
- net DRVEN: now also U2.RD3; no longer IC1.RA0, J1.2
- net GND: now also DBGSER.1, GND@1.P, GND@2.P, GND@3.P, GND@4.P, GND@5.P, GND@6.P, IC1B.+IN, IC1B.-IN, IC1P.V-, PROGVSS.S, U2.VSS@1, U2.VSS@2; no longer IC1.VSS, IC2.GND, J1.1, PROG-3.S, R10.1, R12.1, R15.1, R2.1, R6.1, X1.8, X2.8, X3.8, X4.1, X4.6
- net MCCS: now also U2.RD7; no longer IC1.RA1, J2.1
- net MCINT: no longer IC1.RB3
- net MISO: now also U2.RC5; no longer IC1.RB1, J1.8
- net MOSI: now also U2.RC6; no longer IC1.RA6, J1.6
- net N$10: now also DRV1.!COIL1, M1!C1.P; no longer DRV1.M1B, X1.1
- net N$11: now also DRV1.!COIL2, M1!C2.P; no longer DRV1.M2B, X1.7
- net N$12: now also DRV2.!COIL1, M2!C1.P; no longer DRV2.M1B, X2.1
- net N$13: now also DRV2.COIL2, M2C2.P; no longer DRV2.M2A, X2.2
- net N$14: now also DRV2.!COIL2, M2!C2.P; no longer DRV2.M2B, X2.7
- net N$15: now also DRV2.COIL1, M2C1.P; no longer DRV2.M1A, X2.6
- net N$16: now also DRV3.!COIL1, M3!C1.P; no longer DRV3.M1B, X3.1
- net N$17: now also DRV3.COIL2, M3C2.P; no longer DRV3.M2A, X3.2
- net N$18: now also DRV3.COIL1, M3C1.P; no longer DRV3.M1A, X3.6
- net N$19: now also DRV3.!COIL2, M3!C2.P; no longer DRV3.M2B, X3.7
- net N$20: now also PROGPGD.S, U2.RB7/PGD; no longer IC1.RA5/!MCLR!/VPP, PROG-1.S
- net N$21: now also PROG!MCLR.S, R2.1, U2.RE3/!MCLR; no longer IC1.RB7, PROG-4.S
- net N$22: now also PROGPGC.S, U2.RB6/PGC; no longer IC1.RB6, PROG-5.S
- net N$8: now also DRV1.COIL1, M1C1.P; no longer DRV1.M1A, X1.6
- net N$9: now also DRV1.COIL2, M1C2.P; no longer DRV1.M2A, X1.2
- net REFL1: now also REFL1.P; no longer R2.2, X1.4
- net REFL2: now also REFL2.P; no longer R6.2, X2.4
- net REFL3: now also REFL3.P; no longer R10.2, X3.4
- net REFR1: now also REFR1.P; no longer R4.2, X1.9
- net REFR2: now also REFR2.P; no longer R8.2, X2.9
- net REFR3: now also REFR3.P; no longer R12.2, X3.9
- net SCK: now also U2.RC7; no longer IC1.RB4, J1.7
- net UARTRX: now also RX.P, U2.RD1; no longer IC1.RB2, IC2.RO, JP2.2
- net UARTTX: now also TX.P, U2.RD0; no longer IC1.RB5, IC2.DI, JP1.2
- net VCC: now also VCC@1.P, VCC@2.P, VCC@3.P; no longer R14.2, X4.5, X4.9
Other:
- moved on the sheet: R1, R2, R3, R4, R6, R8
